File: NM_LT.sch (KiCad schematic (older format))
At the start: 43 parts, among them IC1 ATMEGA88-P, P1 CONN_01X02, P2 CONN_01X03, P3 CONN_01X02, Q1 FDS4935A, Q2 µPA2753GR

Commit message: 151127 ERC fin.
Parts:
- removed D7: LED, symbol LED
- removed P2: CONN_01X03, symbol CONN_01X03
- removed P3: CONN_01X02, ~, symbol CONN_01X02
- added P3: CONN_POW, symbol CONN_POW
- added P4: CONN_LS, symbol CONN_LS
- added R23, R24: R, symbol R
- added U1: RPR-220, symbol RPR-220
- gave numbers to parts that had none: 11
Connections:
- net labels added: LED1, LED2, LED3, LED4, LED5, LED6
- wire segments 69 -> 79
- no-connect marks 0 -> 9
Other:
- moved on the sheet: C1, C2

Commit message: 151128 RPR-220 フットプリント作成
Parts:
- C1: footprint (none) -> Capacitors_ThroughHole:C_Axial_D5_L11_P18
- C2, C3: footprint (none) -> Capacitors_ThroughHole:C_Rect_L4_W2.5_P2.5
- IC1: footprint DIL28 -> (none)
- P1, P2: footprint Connect:PINHEAD1-2 -> Pin_Headers:Pin_Header_Angled_1x02
- P3: footprint (none) -> Pin_Headers:Pin_Header_Angled_1x02
- P4: footprint (none) -> Pin_Headers:Pin_Header_Angled_1x03
- Q1, Q2, Q3, Q4: footprint SOP8 -> (none)
Changed lines of the file:
@@
 F 0 "IC1" H 3650 4500 40  0000 L BNN
 F 1 "ATMEGA88-P" H 4850 1850 40  0000 L BNN
-F 2 "DIL28" H 4500 3200 30  0000 C CIN
+F 2 "" H 4500 3200 30  0001 C CIN
 F 3 "" H 4500 3200 60  0000 C CNN
 	1    4500 3200
@@
 F 0 "Q2" H 5500 7125 50  0000 L CNN
 F 1 "µPA2753GR" H 5500 7050 50  0000 L CNN
-F 2 "SOP8" H 5500 6975 50  0000 L CIN
+F 2 "" H 5500 6975 50  0001 L CIN
 F 3 "" H 5300 7050 50  0000 L CNN
 	2    5350 7050
@@
 F 0 "Q2" H 4300 7125 50  0000 L CNN
 F 1 "µPA2753GR" H 4300 7050 50  0000 L CNN
-F 2 "SOP8" H 4300 6975 50  0000 L CIN
+F 2 "" H 4300 6975 50  0001 L CIN
 F 3 "" H 4100 7050 50  0000 L CNN
 	1    4150 7050
@@
 F 0 "Q1" H 4300 6625 50  0000 L CNN
 F 1 "FDS4935A" H 4300 6550 50  0000 L CNN
-F 2 "SOP8" H 4300 6475 50  0000 L CIN
+F 2 "" H 4300 6475 50  0001 L CIN
 F 3 "" H 4100 6550 50  0000 L CNN
 	1    4150 6550
@@
 F 0 "Q1" H 5500 6625 50  0000 L CNN
 F 1 "FDS4935A" H 5500 6550 50  0000 L CNN
-F 2 "SOP8" H 5500 6475 50  0000 L CIN
+F 2 "" H 5500 6475 50  0001 L CIN
 F 3 "" H 5300 6550 50  0000 L CNN
 	2    5350 6550
@@
 F 0 "R6" V 6980 1850 50  0000 C CNN
 F 1 "1k" V 6900 1850 50  0000 C CNN
-F 2 "" V 6830 1850 30  0000 C CNN
+F 2 "" V 6830 1850 30  0001 C CNN
 F 3 "" H 6900 1850 30  0000 C CNN
 	1    6900 1850
@@
 F 0 "C1" H 3075 2300 50  0000 L CNN
 F 1 "CP" H 3075 2100 50  0000 L CNN
-F 2 "" H 3088 2050 30  0000 C CNN
+F 2 "Capacitors_ThroughHole:C_Axial_D5_L11_P18" H 3088 2050 30  0001 C CNN
 F 3 "" H 3050 2200 60  0000 C CNN
 	1    3050 2200
@@
 F 0 "C2" H 3275 2300 50  0000 L CNN
 F 1 "C" H 3275 2100 50  0000 L CNN
-F 2 "" H 3288 2050 30  0000 C CNN
+F 2 "Capacitors_ThroughHole:C_Rect_L4_W2.5_P2.5" H 3288 2050 30  0001 C CNN
 F 3 "" H 3250 2200 60  0000 C CNN
 	1    3250 2200
@@
 F 0 "D2" H 7550 1950 50  0000 C CNN
 F 1 "LED" H 7550 1750 50  0000 C CNN
-F 2 "" H 7550 1850 60  0000 C CNN
+F 2 "" H 7550 1850 60  0001 C CNN
 F 3 "" H 7550 1850 60  0000 C CNN
 	1    7550 1850
@@
 F 0 "R10" V 6980 2250 50  0000 C CNN
 F 1 "1k" V 6900 2250 50  0000 C CNN
-F 2 "" V 6830 2250 30  0000 C CNN
+F 2 "" V 6830 2250 30  0001 C CNN
 F 3 "" H 6900 2250 30  0000 C CNN
 	1    6900 2250
@@
 F 0 "D6" H 7550 2350 50  0000 C CNN
 F 1 "LED" H 7550 2150 50  0000 C CNN
-F 2 "" H 7550 2250 60  0000 C CNN
+F 2 "" H 7550 2250 60  0001 C CNN
 F 3 "" H 7550 2250 60  0000 C CNN
 	1    7550 2250
@@
 F 0 "R7" V 6980 1950 50  0000 C CNN
 F 1 "1k" V 6900 1950 50  0000 C CNN
-F 2 "" V 6830 1950 30  0000 C CNN
+F 2 "" V 6830 1950 30  0001 C CNN
 F 3 "" H 6900 1950 30  0000 C CNN
 	1    6900 1950
@@
 F 0 "R2" V 3680 7100 50  0000 C CNN
 F 1 "R" V 3600 7100 50  0000 C CNN
-F 2 "" V 3530 7100 30  0000 C CNN
+F 2 "" V 3530 7100 30  0001 C CNN
 F 3 "" H 3600 7100 30  0000 C CNN
 	1    3600 7100
@@
 F 0 "R4" V 3980 7250 50  0000 C CNN
 F 1 "R" V 3900 7250 50  0000 C CNN
-F 2 "" V 3830 7250 30  0000 C CNN
+F 2 "" V 3830 7250 30  0001 C CNN
 F 3 "" H 3900 7250 30  0000 C CNN
 	1    3900 7250
@@
 F 0 "R14" V 5980 7100 50  0000 C CNN
 F 1 "R" V 5900 7100 50  0000 C CNN
-F 2 "" V 5830 7100 30  0000 C CNN
+F 2 "" V 5830 7100 30  0001 C CNN
 F 3 "" H 5900 7100 30  0000 C CNN
 	1    5900 7100
@@
 F 0 "R12" V 5680 7250 50  0000 C CNN
 F 1 "R" V 5600 7250 50  0000 C CNN
-F 2 "" V 5530 7250 30  0000 C CNN
+F 2 "" V 5530 7250 30  0001 C CNN
 F 3 "" H 5600 7250 30  0000 C CNN
 	1    5600 7250
@@
 F 0 "P1" H 4750 6750 50  0000 C CNN
 F 1 "CONN_01X02" V 4850 6600 50  0000 C CNN
-F 2 "Connect:PINHEAD1-2" H 4750 6600 60  0000 C CNN
+F 2 "Pin_Headers:Pin_Header_Angled_1x02" H 4750 6600 60  0001 C CNN
 F 3 "" H 4750 6600 60  0001 C CNN
 	1    4750 6600
@@
 F 0 "R1" V 3680 6600 50  0000 C CNN
 F 1 "R" V 3600 6600 50  0000 C CNN
-F 2 "" V 3530 6600 30  0000 C CNN
+F 2 "" V 3530 6600 30  0001 C CNN
 F 3 "" H 3600 6600 30  0000 C CNN
 	1    3600 6600
@@
 F 0 "R3" V 3980 6350 50  0000 C CNN
 F 1 "R" V 3900 6350 50  0000 C CNN
-F 2 "" V 3830 6350 30  0000 C CNN
+F 2 "" V 3830 6350 30  0001 C CNN
 F 3 "" H 3900 6350 30  0000 C CNN
 	1    3900 6350
@@
 F 0 "R13" V 5980 6600 50  0000 C CNN
 F 1 "R" V 5900 6600 50  0000 C CNN
-F 2 "" V 5830 6600 30  0000 C CNN
+F 2 "" V 5830 6600 30  0001 C CNN
 F 3 "" H 5900 6600 30  0000 C CNN
 	1    5900 6600
@@
 F 0 "R11" V 5680 6350 50  0000 C CNN
 F 1 "R" V 5600 6350 50  0000 C CNN
-F 2 "" V 5530 6350 30  0000 C CNN
+F 2 "" V 5530 6350 30  0001 C CNN
 F 3 "" H 5600 6350 30  0000 C CNN
 	1    5600 6350
@@
 F 0 "D3" H 7550 2050 50  0000 C CNN
 F 1 "LED" H 7550 1850 50  0000 C CNN
-F 2 "" H 7550 1950 60  0000 C CNN
+F 2 "" H 7550 1950 60  0001 C CNN
 F 3 "" H 7550 1950 60  0000 C CNN
 	1    7550 1950
@@
 F 0 "R9" V 6980 2150 50  0000 C CNN
 F 1 "1k" V 6900 2150 50  0000 C CNN
-F 2 "" V 6830 2150 30  0000 C CNN
+F 2 "" V 6830 2150 30  0001 C CNN
 F 3 "" H 6900 2150 30  0000 C CNN
 	1    6900 2150
@@
 F 0 "D5" H 7550 2250 50  0000 C CNN
 F 1 "LED" H 7550 2050 50  0000 C CNN
-F 2 "" H 7550 2150 60  0000 C CNN
+F 2 "" H 7550 2150 60  0001 C CNN
 F 3 "" H 7550 2150 60  0000 C CNN
 	1    7550 2150
@@
 F 0 "R5" V 6980 1750 50  0000 C CNN
 F 1 "1k" V 6900 1750 50  0000 C CNN
-F 2 "" V 6830 1750 30  0000 C CNN
+F 2 "" V 6830 1750 30  0001 C CNN
 F 3 "" H 6900 1750 30  0000 C CNN
 	1    6900 1750
@@
 F 0 "D1" H 7550 1850 50  0000 C CNN
 F 1 "LED" H 7550 1650 50  0000 C CNN
-F 2 "" H 7550 1750 60  0000 C CNN
+F 2 "" H 7550 1750 60  0001 C CNN
 F 3 "" H 7550 1750 60  0000 C CNN
 	1    7550 1750
@@
 F 0 "R8" V 6980 2050 50  0000 C CNN
 F 1 "1k" V 6900 2050 50  0000 C CNN
-F 2 "" V 6830 2050 30  0000 C CNN
+F 2 "" V 6830 2050 30  0001 C CNN
 F 3 "" H 6900 2050 30  0000 C CNN
 	1    6900 2050
@@
 F 0 "D4" H 7550 2150 50  0000 C CNN
 F 1 "LED" H 7550 1950 50  0000 C CNN
-F 2 "" H 7550 2050 60  0000 C CNN
+F 2 "" H 7550 2050 60  0001 C CNN
 F 3 "" H 7550 2050 60  0000 C CNN
 	1    7550 2050
@@
 F 0 "C3" H 3525 2900 50  0000 L CNN
 F 1 "C" H 3525 2700 50  0000 L CNN
-F 2 "" H 3538 2650 30  0000 C CNN
+F 2 "Capacitors_ThroughHole:C_Rect_L4_W2.5_P2.5" H 3538 2650 30  0001 C CNN
 F 3 "" H 3500 2800 60  0000 C CNN
 	1    3500 2800
@@
 F 0 "Q4" H 5500 5925 50  0000 L CNN
 F 1 "µPA2753GR" H 5500 5850 50  0000 L CNN
-F 2 "SOP8" H 5500 5775 50  0000 L CIN
+F 2 "" H 5500 5775 50  0001 L CIN
 F 3 "" H 5300 5850 50  0000 L CNN
 	2    5350 5850
@@
 F 0 "Q4" H 4300 5925 50  0000 L CNN
 F 1 "µPA2753GR" H 4300 5850 50  0000 L CNN
-F 2 "SOP8" H 4300 5775 50  0000 L CIN
+F 2 "" H 4300 5775 50  0001 L CIN
 F 3 "" H 4100 5850 50  0000 L CNN
 	1    4150 5850
@@
 F 0 "Q3" H 4300 5425 50  0000 L CNN
 F 1 "FDS4935A" H 4300 5350 50  0000 L CNN
-F 2 "SOP8" H 4300 5275 50  0000 L CIN
+F 2 "" H 4300 5275 50  0001 L CIN
 F 3 "" H 4100 5350 50  0000 L CNN
 	1    4150 5350
@@
 F 0 "Q3" H 5500 5425 50  0000 L CNN
 F 1 "FDS4935A" H 5500 5350 50  0000 L CNN
-F 2 "SOP8" H 5500 5275 50  0000 L CIN
+F 2 "" H 5500 5275 50  0001 L CIN
 F 3 "" H 5300 5350 50  0000 L CNN
 	2    5350 5350
@@
 F 0 "R16" V 3680 5900 50  0000 C CNN
 F 1 "R" V 3600 5900 50  0000 C CNN
-F 2 "" V 3530 5900 30  0000 C CNN
+F 2 "" V 3530 5900 30  0001 C CNN
 F 3 "" H 3600 5900 30  0000 C CNN
 	1    3600 5900
@@
 F 0 "R18" V 3980 6050 50  0000 C CNN
 F 1 "R" V 3900 6050 50  0000 C CNN
-F 2 "" V 3830 6050 30  0000 C CNN
+F 2 "" V 3830 6050 30  0001 C CNN
 F 3 "" H 3900 6050 30  0000 C CNN
 	1    3900 6050
@@
 F 0 "R22" V 5980 5900 50  0000 C CNN
 F 1 "R" V 5900 5900 50  0000 C CNN
-F 2 "" V 5830 5900 30  0000 C CNN
+F 2 "" V 5830 5900 30  0001 C CNN
 F 3 "" H 5900 5900 30  0000 C CNN
 	1    5900 5900
@@
 F 0 "R20" V 5680 6050 50  0000 C CNN
 F 1 "R" V 5600 6050 50  0000 C CNN
-F 2 "" V 5530 6050 30  0000 C CNN
+F 2 "" V 5530 6050 30  0001 C CNN
 F 3 "" H 5600 6050 30  0000 C CNN
 	1    5600 6050
@@
 F 0 "P2" H 4750 5550 50  0000 C CNN
 F 1 "CONN_01X02" V 4850 5400 50  0000 C CNN
-F 2 "Connect:PINHEAD1-2" H 4750 5400 60  0000 C CNN
+F 2 "Pin_Headers:Pin_Header_Angled_1x02" H 4750 5400 60  0001 C CNN
 F 3 "" H 4750 5400 60  0001 C CNN
 	1    4750 5400
@@
 F 0 "R15" V 3680 5400 50  0000 C CNN
 F 1 "R" V 3600 5400 50  0000 C CNN
-F 2 "" V 3530 5400 30  0000 C CNN
+F 2 "" V 3530 5400 30  0001 C CNN
 F 3 "" H 3600 5400 30  0000 C CNN
 	1    3600 5400
@@
 F 0 "R17" V 3980 5150 50  0000 C CNN
 F 1 "R" V 3900 5150 50  0000 C CNN
-F 2 "" V 3830 5150 30  0000 C CNN
+F 2 "" V 3830 5150 30  0001 C CNN
 F 3 "" H 3900 5150 30  0000 C CNN
 	1    3900 5150
@@
 F 0 "R21" V 5980 5400 50  0000 C CNN
 F 1 "R" V 5900 5400 50  0000 C CNN
-F 2 "" V 5830 5400 30  0000 C CNN
+F 2 "" V 5830 5400 30  0001 C CNN
 F 3 "" H 5900 5400 30  0000 C CNN
 	1    5900 5400
@@
 F 0 "R19" V 5680 5150 50  0000 C CNN
 F 1 "R" V 5600 5150 50  0000 C CNN
-F 2 "" V 5530 5150 30  0000 C CNN
+F 2 "" V 5530 5150 30  0001 C CNN
 F 3 "" H 5600 5150 30  0000 C CNN
 	1    5600 5150
@@
 F 0 "U1" H 7600 5200 50  0000 L CNN
 F 1 "RPR-220" H 7650 4800 50  0000 L CNN
-F 2 "" H 7600 4800 50  0000 L CIN
+F 2 "" H 7600 4800 50  0001 L CIN
 F 3 "" H 7800 5000 50  0000 L CNN
 	1    7800 5000
@@
 F 0 "R23" V 7580 4750 50  0000 C CNN
 F 1 "R" V 7500 4750 50  0000 C CNN
-F 2 "" V 7430 4750 30  0000 C CNN
+F 2 "" V 7430 4750 30  0001 C CNN
 F 3 "" H 7500 4750 30  0000 C CNN
 	1    7500 4750
@@
 F 0 "R24" V 8180 5250 50  0000 C CNN
 F 1 "R" V 8100 5250 50  0000 C CNN
-F 2 "" V 8030 5250 30  0000 C CNN
+F 2 "" V 8030 5250 30  0001 C CNN
 F 3 "" H 8100 5250 30  0000 C CNN
 	1    8100 5250
@@
 F 0 "P4" H 8450 5500 50  0000 C CNN
 F 1 "CONN_LS" V 8550 5300 50  0000 C CNN
-F 2 "" H 8450 5300 60  0000 C CNN
+F 2 "Pin_Headers:Pin_Header_Angled_1x03" H 8450 5300 60  0001 C CNN
 F 3 "" H 8450 5300 60  0000 C CNN
 	1    8450 5300
@@
 F 0 "P3" H 2450 2400 50  0000 C CNN
 F 1 "CONN_POW" V 2550 2250 50  0000 C CNN
-F 2 "" H 2450 2250 60  0000 C CNN
+F 2 "Pin_Headers:Pin_Header_Angled_1x02" H 2450 2250 60  0001 C CNN
 F 3 "" H 2450 2250 60  0000 C CNN
 	1    2450 2250

Commit message: 151206 FootPrint 40% fin.
Parts:
- D1, D2, D3, D4, D5, D6: footprint (none) -> LEDs:LED-3MM
- IC1: footprint (none) -> Housings_DIP:DIP-28_W7.62mm_LongPads
Changed lines of the file:
@@
 F 0 "IC1" H 3650 4500 40  0000 L BNN
 F 1 "ATMEGA88-P" H 4850 1850 40  0000 L BNN
-F 2 "" H 4500 3200 30  0001 C CIN
+F 2 "Housings_DIP:DIP-28_W7.62mm_LongPads" H 4500 3200 30  0001 C CIN
 F 3 "" H 4500 3200 60  0000 C CNN
 	1    4500 3200
@@
 F 0 "D2" H 7550 1950 50  0000 C CNN
 F 1 "LED" H 7550 1750 50  0000 C CNN
-F 2 "" H 7550 1850 60  0001 C CNN
+F 2 "LEDs:LED-3MM" H 7550 1850 60  0001 C CNN
 F 3 "" H 7550 1850 60  0000 C CNN
 	1    7550 1850
@@
 F 0 "D6" H 7550 2350 50  0000 C CNN
 F 1 "LED" H 7550 2150 50  0000 C CNN
-F 2 "" H 7550 2250 60  0001 C CNN
+F 2 "LEDs:LED-3MM" H 7550 2250 60  0001 C CNN
 F 3 "" H 7550 2250 60  0000 C CNN
 	1    7550 2250
@@
 F 0 "D3" H 7550 2050 50  0000 C CNN
 F 1 "LED" H 7550 1850 50  0000 C CNN
-F 2 "" H 7550 1950 60  0001 C CNN
+F 2 "LEDs:LED-3MM" H 7550 1950 60  0001 C CNN
 F 3 "" H 7550 1950 60  0000 C CNN
 	1    7550 1950
@@
 F 0 "D5" H 7550 2250 50  0000 C CNN
 F 1 "LED" H 7550 2050 50  0000 C CNN
-F 2 "" H 7550 2150 60  0001 C CNN
+F 2 "LEDs:LED-3MM" H 7550 2150 60  0001 C CNN
 F 3 "" H 7550 2150 60  0000 C CNN
 	1    7550 2150
@@
 F 0 "D1" H 7550 1850 50  0000 C CNN
 F 1 "LED" H 7550 1650 50  0000 C CNN
-F 2 "" H 7550 1750 60  0001 C CNN
+F 2 "LEDs:LED-3MM" H 7550 1750 60  0001 C CNN
 F 3 "" H 7550 1750 60  0000 C CNN
 	1    7550 1750
@@
 F 0 "D4" H 7550 2150 50  0000 C CNN
 F 1 "LED" H 7550 1950 50  0000 C CNN
-F 2 "" H 7550 2050 60  0001 C CNN
+F 2 "LEDs:LED-3MM" H 7550 2050 60  0001 C CNN
 F 3 "" H 7550 2050 60  0000 C CNN
 	1    7550 2050

Commit message: 151213 fix two compornent
Parts:
- R1, R10, R11, R12, R13, R14, R15, R16, R17, R18, R19, R2, R20, R21, R22, R23, R24, R3, R4, R5, R6, R7, R8, R9: footprint (none) -> Resistors_ThroughHole:Resistor_Horizontal_RM25mm
Connections:
- net at P1.2 (P2), Q2.5 (D): now also Q1.5 (D), Q1.6 (D), Q2.6 (D); no longer Q1.3 (S)
- net at P1.1 (P1), Q2.7 (D): now also Q1.7 (D), Q1.8 (D), Q2.8 (D); no longer Q1.1 (S)
- net at P2.2 (P2), Q4.5 (D): now also Q3.5 (D), Q3.6 (D), Q4.6 (D); no longer Q3.3 (S)
- net at P2.1 (P1), Q4.7 (D): now also Q3.7 (D), Q3.8 (D), Q4.8 (D); no longer Q3.1 (S)
- new net: Q1.1 (S), R3.1
- new net: Q1.3 (S), R11.1
- new net: Q3.1 (S), R17.1
- new net: Q3.3 (S), R19.1
